File: elec/layout/default.kicad_pcb (KiCad board)
At the start: 2 copper layers, 45 x 53 mm, 40 parts

Commit message: Add pcb files
Parts:
- removed C10, C11, C12, C13, C14, C15, C16, C7, C8, C9: , atopile:C_0201_0603Metric
- removed R10, R9: , atopile:R_0201_0603Metric
- removed R11, R5, R6, R7, R8: , atopile:R_0402_1005Metric
- added C19: 100nF ±10% 16V X7R, atopile:C0402-b3ef17, F.Cu at (-3.35, 0.00)
- added JP1: , NetTie:NetTie-2_SMD_Pad0.5mm, F.Cu at (39.8, 21.2)
- added R16: 470Ω ±1% 62.5mW, atopile:R0402-56259e, F.Cu at (-3.12, 0.95)
- added R17: 470Ω ±1% 62.5mW, atopile:R0402-56259e, F.Cu at (-5.36, -0.95)
- added U3: , atopile:SOT-23-6_L2.9-W1.6-P0.95-LS2.8-BR-bfc73b, F.Cu at (27.6, 24.0)
- C1: value 1µF ±10% 50V X5R -> 1µF ±10% 25V X5R; footprint atopile:C0603-bd72f6 -> atopile:C0402-b3ef17
- C17: value 10nF ±1% 50V C0G -> 47pF ±1% 50V C0G; footprint atopile:C0805-3b2e55 -> atopile:C0402-b3ef17
- C18: value 22nF ±1% 50V -> 22nF ±10% 50V X7R; footprint atopile:C0805-3b2e55 -> atopile:C0402-b3ef17
- C2, C3: value 10µF ±10% 10V X5R -> 10µF ±10% 35V X7R; footprint atopile:C0603-bd72f6 -> atopile:C1210-c93926
- MOD1: footprint ki-lime-pi-pico:RaspberryPi_Pico_Common_THT -> atopile:COMM-SMD_RP2040-ZERO-70d39b
- R12: value 10kΩ ±1% 100mW -> 49.9Ω ±1% 62.5mW; footprint atopile:R0603-ebcab9 -> atopile:R0402-56259e
- R13: value 49.9Ω ±1% 100mW -> 10kΩ ±1% 62.5mW; footprint atopile:R0603-ebcab9 -> atopile:R0402-56259e
- R14: value 0Ω 100mW -> 10kΩ ±1% 62.5mW; footprint atopile:R0603-ebcab9 -> atopile:R0402-56259e
- moved C17 356.2 mm to (45.0, 24.5), turned to 90 degrees
- moved C18 330.6 mm to (40.8, 25.0), turned to 90 degrees
- moved R12 167.2 mm to (45.0, 22.0), turned to -90 degrees
- moved R13 149.2 mm to (43.8, 24.5), turned to -90 degrees
- moved J3 85.9 mm to (47.0, 43.5), turned to 0 degrees
- moved R14 72.9 mm to (44.2, 26.5), turned to 180 degrees
- moved J4 71.5 mm to (65.0, 43.5)
- moved C6 68.6 mm to (54.0, 29.2), turned to -90 degrees
- moved C5 66.9 mm to (50.0, 35.2), turned to 90 degrees
- moved C4 63.3 mm to (50.0, 29.2), turned to -90 degrees
- moved U2 58.2 mm to (44.0, 32.2), turned to -90 degrees
- moved MOD1 57.5 mm to (12.0, 40.0)
- moved C2 54.2 mm to (38.0, 35.2), turned to 90 degrees
- moved R4 51.6 mm to (42.0, 25.0), turned to 90 degrees
- moved C3 49.4 mm to (38.0, 29.2), turned to -90 degrees
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Connections:
- net contact[10] renamed mcu-line-5
- net contact[11] renamed mcu-line-8
- net contact[13] renamed mcu-line-16
- net contact[15] renamed mcu-line-10
- net contact[16] renamed mcu-line-7
- net contact[19] renamed mcu-line-3
- net mcu-contact[0] renamed mcu-line-4
- net mcu-contact[0]-1 renamed mcu-hv
- net mcu-contact[14] renamed mcu-line-13
- net mcu-contact[18]-1 renamed mcu-line-11
- net mcu-contact[1]-1 renamed mcu-line-12
- net mcu-contact[6] renamed mcu-line-17
- net mcu-contact[8] renamed mcu-line-9
- net pd_power_supply.usb_pr_trigger.power_good_indicator.led-cathode renamed cathode
- C1 pad 2: gnd-1 -> gnd
- C17 pad 1: feedback -> dcdc_module-line-2
- C17 pad 2: unnamed[1] -> dcdc_module.output_voltage_feedback-hv-1
- C2 pad 2: gnd-1 -> gnd
- C3 pad 2: gnd-1 -> gnd
- C4 pad 2: gnd-1 -> gnd
- C5 pad 2: gnd-1 -> gnd
- C6 pad 2: gnd-1 -> gnd
- J3 pad 1: hv-1 -> hv-2
- J3 pad 2: gnd-1 -> gnd
- J4 pad 1: hv-1 -> hv-2
- J4 pad 2: gnd-1 -> gnd
- J4 pad 3: clock -> data
- J4 pad 4: data -> clock
- J5 pad A1: gnd-1 -> gnd
- J5 pad A12: gnd-1 -> gnd
- J5 pad B1: gnd-1 -> gnd
- J5 pad B12: gnd-1 -> gnd
- MOD1 pad 10: mcu-contact[9]-1 -> mcu-line-2
- MOD1 pad 13: gnd -> mcu-line-6
- MOD1 pad 18: gnd -> mcu-line
- MOD1 pad 22: mcu-contact[1] -> gnd
- MOD1 pad 23: gnd -> mcu-hv-1
- MOD1 pad 3: gnd -> line-1
- MOD1 pad 4: clock -> line
- MOD1 pad 5: data -> mcu-line-15
- MOD1 pad 6: mcu-contact[5] -> mcu-line-1
- MOD1 pad 8: gnd -> mcu-line-14
- R12 pad 1: feedback -> hv-1
- R12 pad 2: dcdc_module-gnd -> dcdc_module.output_voltage_feedback-hv
- R13 pad 1: unnamed[1] -> dcdc_module.output_voltage_feedback-hv-1
- R13 pad 2: hv-1 -> dcdc_module-line-2
- R14 pad 1: feedback -> dcdc_module-line-2
- R14 pad 2: unnamed[1] -> dcdc_module-gnd
- R4 pad 1: dcdc_module-line -> dcdc_module-line-1
- U1 pad 11: gnd-1 -> gnd
- U1 pad 2: pd_power_supply.usb_pr_trigger.controller-line-1 -> pd_power_supply.usb_pr_trigger.controller-line
- U1 pad 9: pd_power_supply.usb_pr_trigger.controller-line -> pd_power_supply.usb_pr_trigger.controller-line-1
- U2 pad 13: gnd-1 -> gnd
- U2 pad 14: gnd-1 -> gnd
- U2 pad 15: gnd-1 -> gnd
- U2 pad 17: gnd-1 -> gnd
- U2 pad 18: gnd-1 -> gnd
- U2 pad 19: gnd-1 -> gnd
- U2 pad 3: dcdc_module-line-1 -> dcdc_module-line
- U2 pad 4: feedback -> dcdc_module-line-2
- U2 pad 6: dcdc_module-line -> dcdc_module-line-1
Routing:
- net led_buffer-line: track 0.00 -> 64.2 mm
- net hv-1: track 0.00 -> 56.3 mm, vias 21 -> 41
- net led_buffer-line-1: track 0.00 -> 46.7 mm
- net vbus: track 37.3 -> 24.5 mm, vias 28 -> 3
- net dcdc_module-line-2: track 0.00 -> 6.61 mm
- net pd_power_supply-gnd: track 8.83 -> 2.85 mm
- net frequency_mode: track 0.00 -> 5.45 mm
- net soft_start: track 0.00 -> 5.33 mm
- net dcdc_module-line-1: track 0.00 -> 5.14 mm
- net dcdc_module-line: track 2.05 -> 6.17 mm
- net sbu2: track 0.00 -> 2.82 mm, vias 0 -> 2
- net dcdc_module-gnd: track 0.00 -> 1.55 mm
- net pd_power_supply-line: vias 2 -> 23
- net mcu-line-16: vias 4 -> 0
- net mcu-contact[6]-1: vias 2 -> 0
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- added copper zone on F.Cu, net dcdc_module-gnd
- added copper zone on B.Cu, net gnd
- added copper zone on F.Cu, net gnd
- removed copper zone on B.Cu, net gnd-1
- removed copper zone on F.Cu, net gnd-1
Other:
- board size 45 x 53 mm -> 75 x 33 mm
