File: elec/layout/tpsm86837rcgr/tpsm86837rcgr.kicad_pcb (KiCad board)
At the start: 2 copper layers, 1 part

Commit message: Add pcb files
Connections:
- U1 pad 13: gnd -> gnd-1
- U1 pad 14: gnd -> gnd-1
- U1 pad 15: gnd -> gnd-1
- U1 pad 17: gnd -> gnd-1
- U1 pad 18: gnd -> gnd-1
- U1 pad 19: gnd -> gnd-1
- U1 pad 4: feedback -> line
- U1 pad 5: gnd-1 -> gnd
- U1 pad 6: line -> line-2
Changed lines of the file:
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@@
             (outputdirectory "")))
     (net 0 "")
-    (net 1 "feedback")
-    (net 2 "line")
+    (net 1 "line")
+    (net 2 "line-2")
     (net 3 "line-1")
-    (net 4 "gnd")
-    (net 5 "gnd-1")
+    (net 4 "gnd-1")
+    (net 5 "gnd")
     (net 6 "footprint.pins[2].net-net")
     (net 7 "hv")
@@
             (layers "F.Cu" "F.Paste" "F.Mask")
             (remove_unused_layers no)
-            (net 1 "feedback"))
+            (net 1 "line"))
         (pad "5" smd rect
             (at -2.2 0.25 0)
@@
             (layers "F.Cu" "F.Paste" "F.Mask")
             (remove_unused_layers no)
-            (net 5 "gnd-1"))
+            (net 5 "gnd"))
         (pad "6" smd rect
             (at -2.2 0.75 0)
@@
             (layers "F.Cu" "F.Paste" "F.Mask")
             (remove_unused_layers no)
-            (net 2 "line"))
+            (net 2 "line-2"))
         (pad "7" smd rect
             (at -2.2 1.25 0)
@@
             (layers "F.Cu" "F.Paste" "F.Mask")
             (remove_unused_layers no)
-            (net 4 "gnd"))
+            (net 4 "gnd-1"))
         (pad "14" smd rect
             (at 2.2 -0.75 0)
@@
             (layers "F.Cu" "F.Paste" "F.Mask")
             (remove_unused_layers no)
-            (net 4 "gnd"))
+            (net 4 "gnd-1"))
         (pad "15" smd rect
             (at 2.2 -1.25 0)
@@
             (layers "F.Cu" "F.Paste" "F.Mask")
             (remove_unused_layers no)
-            (net 4 "gnd"))
+            (net 4 "gnd-1"))
         (pad "16" smd rect
             (at 2.1 -2.15 0)
@@
             (layers "F.Cu" "F.Paste" "F.Mask")
             (remove_unused_layers no)
-            (net 4 "gnd"))
+            (net 4 "gnd-1"))
         (pad "18" smd rect
             (at 0 0 0)
@@
             (layers "F.Cu" "F.Paste" "F.Mask")
             (remove_unused_layers no)
-            (net 4 "gnd"))
+            (net 4 "gnd-1"))
         (pad "19" smd rect
             (at 0 1.05 0)
@@
             (layers "F.Cu" "F.Paste" "F.Mask")
             (remove_unused_layers no)
-            (net 4 "gnd"))))
+            (net 4 "gnd-1"))))
