File: elec/layout/usb_power_source/usb_power_source.kicad_pcb (KiCad board)
At the start: 2 copper layers, 7 parts

Commit message: Change PCB layout
Connections:
- U1 pad 3: usb_pr_trigger.controller-signal-2 -> usb_pr_trigger.controller-signal
- U1 pad 9: usb_pr_trigger.controller-signal -> usb_pr_trigger.controller-signal-2
Changed lines of the file:
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@@
 	(net 3 "cc[0]")
 	(net 4 "usb_pr_trigger.controller-signal-1")
-	(net 5 "usb_pr_trigger.controller-signal-2")
+	(net 5 "usb_pr_trigger.controller-signal")
 	(net 6 "cathode")
-	(net 7 "usb_pr_trigger.controller-signal")
+	(net 7 "usb_pr_trigger.controller-signal-2")
 	(net 8 "hv")
 	(net 9 "usb_pr_trigger-hv")
@@
 			(size 1.5 0.6)
 			(layers "F.Cu" "F.Paste" "F.Mask")
-			(net 5 "usb_pr_trigger.controller-signal-2")
+			(net 5 "usb_pr_trigger.controller-signal")
 		)
 		(pad "4" smd rect
@@
 			(size 1.5 0.6)
 			(layers "F.Cu" "F.Paste" "F.Mask")
-			(net 7 "usb_pr_trigger.controller-signal")
+			(net 7 "usb_pr_trigger.controller-signal-2")
 		)
 		(pad "10" smd rect
@@
 		(layers "F&B.Cu")
 		(hatch edge 0.5)
+		(priority 1)
 		(connect_pads
 			(clearance 0.25)

Commit message: Add LED buffer, change DCDC func to params, layout
Parts:
- C1: value 100nF ±10% 50V X7R -> 1µF ±10% 50V X5R
Connections:
- net signal renamed line
- net signal-1 renamed line-1
- net usb_pr_trigger-signal renamed usb_pr_trigger-line
- net usb_pr_trigger.controller-signal renamed usb_pr_trigger.controller-line
- net usb_pr_trigger.controller-signal-1 renamed usb_pr_trigger.controller-line-1
- net usb_pr_trigger.controller-signal-2 renamed usb_pr_trigger.controller-line-2

Commit message: Add pcb files
Parts:
- removed the C1 at (-3.75, -9.50)
- added C1: 10µF ±10% 35V X7R, atopile:C1210-c93926, F.Cu at (-6.00, 3.00)
- added C1: 1µF ±10% 25V X5R, atopile:C0402-b3ef17, F.Cu at (20.0, -5.00)
- added C2: 10µF ±10% 35V X7R, atopile:C1210-c93926, F.Cu at (-6.00, -3.00)
- added C5: 22µF ±10% 25V X7R, atopile:C1210-c93926, F.Cu at (10.0, -3.00)
- added C6: 47pF ±1% 50V C0G, atopile:C0402-b3ef17, F.Cu at (1.00, -7.75)
- added C7: 22nF ±10% 50V X7R, atopile:C0402-b3ef17, F.Cu at (-3.25, -7.25)
- added JP1: , NetTie:NetTie-2_SMD_Pad0.5mm, F.Cu at (-4.25, -11.0)
- added R4: 10kΩ ±1% 62.5mW, atopile:R0402-56259e, F.Cu at (0.25, -5.75)
- moved R3 73.8 mm to (70.0, -5.00), turned to 0 degrees
- moved J1 60.2 mm to (60.0, -5.00)
- moved R2 51.1 mm to (50.0, -5.00), turned to 0 degrees
- moved U1 40.3 mm to (40.0, -5.00)
- moved D1 26.7 mm to (30.0, -5.00), turned to 0 degrees
- moved R1 10.4 mm to (10.0, -5.00), turned to 0 degrees
Routing:
- net hv: track 37.3 -> 0.00 mm, vias 4 -> 24
- net (no net): track 0.00 -> 25.0 mm, vias 0 -> 118
- net cc[0]: track 14.5 -> 0.00 mm, vias 2 -> 0
- net cc[1]: track 13.8 -> 0.00 mm, vias 2 -> 0
- net line: track 9.83 -> 0.00 mm, vias 2 -> 0
- net gnd-1: track 8.83 -> 1.55 mm
- net soft_start: track 0.00 -> 5.33 mm
- net usb_pr_trigger-hv: track 3.55 -> 0.00 mm
- net output_voltage_feedback-hv: track 0.00 -> 2.82 mm
- net usb_pr_trigger-line: track 1.75 -> 0.00 mm
- net cathode: track 1.70 -> 0.00 mm
- net line-1: track 6.72 -> 6.17 mm
- net gnd: vias 2 -> 0
- added copper zone on B.Cu, net (none)
- added copper zone on F.Cu, net (none)
- added copper zone on F.Cu, net gnd-1
- added copper zone on B.Cu, net hv
- added copper zone on F.Cu, net hv
- removed copper zone on B.Cu, net gnd
- removed copper zone on F.Cu, net gnd
